File: 6key/pcb.sch (KiCad schematic (older format))
At the start: 13 parts, among them K0 KEYSW, K1 KEYSW, K2 KEYSW, K3 KEYSW, K4 KEYSW, K5 KEYSW, U1 ProMicro

Commit message: shift reg arduino, 2x3 rgb pcb
Parts:
- added LED1, LED2, LED3, LED4, LED5, LED6: LED_CRGB, LED_THT:LED_D5.0mm-4_RGB_NO_CASE, symbol Device:LED_CRGB
- added Q1, Q2: BF244A, Package_TO_SOT_THT:TO-92_Inline, symbol Transistor_FET:BF244A
- added R1, R2, R3, R4, R5, R6, R7, R8, R9: R, Resistor_THT:R_Axial_DIN0207_L6.3mm_D2.5mm_P7.62mm_Horizontal, symbol Device:R
- D1: renamed from D0; footprint Diode_THT:D_T-1_P10.16mm_Horizontal -> Diode_THT:D_T-1_P5.08mm_Horizontal
- D2: renamed from D3; footprint Diode_THT:D_T-1_P10.16mm_Horizontal -> Diode_THT:D_T-1_P5.08mm_Horizontal
- D3: renamed from D1; footprint Diode_THT:D_T-1_P10.16mm_Horizontal -> Diode_THT:D_T-1_P5.08mm_Horizontal
- D4: footprint Diode_THT:D_T-1_P10.16mm_Horizontal -> Diode_THT:D_T-1_P5.08mm_Horizontal
- D5: renamed from D2; footprint Diode_THT:D_T-1_P10.16mm_Horizontal -> Diode_THT:D_T-1_P5.08mm_Horizontal
- D6: renamed from D5; footprint Diode_THT:D_T-1_P10.16mm_Horizontal -> Diode_THT:D_T-1_P5.08mm_Horizontal
- renumbered K0 to K1, K3 to K2, K1 to K3, K2 to K5, K5 to K6
Connections:
- net GND: now also Q1.3 (S), Q2.3 (S)
- net col1: now also U1.16 (B1); no longer U1.11 (B4)
- net col2: now also U1.19 (F5); no longer U1.12 (B5)
- net row0: now also U1.20 (F4), Q1.2 (G); no longer U1.8 (C6)
- net row1: now also U1.13 (B6), Q2.2 (G); no longer U1.9 (D7)
- net led1r: now reaches U1.14 (B2)
- net led1r: now also R4.1
- net led1g: now reaches U1.15 (B3)
- net led1g: now also R5.1
- net led2g: now reaches U1.17 (F7)
- net led2g: now also R8.1
- net led2r: now reaches U1.18 (F6)
- net led2r: now also R7.1
- net led0r: now reaches U1.7 (D4)
- net led0r: now also R1.1
- new net: LED1.1 (K), LED3.1 (K), LED5.1 (K), Q1.1 (D)
- new net: LED1.2 (RA), LED2.2 (RA), R1.2
- new net: LED1.3 (GA), LED2.3 (GA), R2.2
- new net: LED1.4 (BA), LED2.4 (BA), R3.2
- new net: LED5.2 (RA), LED6.2 (RA), R7.2
- new net: LED5.3 (GA), LED6.3 (GA), R8.2
- new net: LED5.4 (BA), LED6.4 (BA), R9.2
- new net: LED3.2 (RA), LED4.2 (RA), R4.2
- new net: LED3.3 (GA), LED4.3 (GA), R5.2
- new net: LED3.4 (BA), LED4.4 (BA), R6.2
- new net: LED2.1 (K), LED4.1 (K), LED6.1 (K), Q2.1 (D)
- new net led0b: R3.1, U1.9 (D7)
- new net led0g: R2.1, U1.8 (C6)
- new net led1b: R6.1, U1.11 (B4)
- new net led2b: R9.1, U1.12 (B5)
- no-connect marks 0 -> 7
Other:
- moved on the sheet: D1, D2, D3, D4, D5, D6, K1, K2, K3, K4, K5, K6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
