File: kicad/keyboard/keyboard.kicad_pcb (KiCad board)
At the start: 2 copper layers, 285 x 94.6 mm, 132 parts, among them K0 KEYSW, K1 KEYSW, K10 KEYSW, K11 KEYSW, K12 KEYSW, K13 KEYSW, K14 KEYSW, K15 KEYSW, K16 KEYSW, K17 KEYSW, K18 KEYSW, K19 KEYSW, K2 KEYSW, K20 KEYSW, K21 KEYSW, K22 KEYSW, K23 KEYSW, K24 KEYSW, K25 KEYSW, K26 KEYSW, K27 KEYSW, K28 KEYSW, K29 KEYSW, K3 KEYSW, K30 KEYSW, K31 KEYSW, K32 KEYSW, K33 KEYSW, K34 KEYSW, K35 KEYSW, K36 KEYSW, K37 KEYSW, K38 KEYSW, K39 KEYSW, K4 KEYSW, K40 KEYSW, K41 KEYSW, K42 KEYSW, K43 KEYSW, K44 KEYSW, K45 KEYSW, K46 KEYSW, K47 KEYSW, K48 KEYSW, K49 KEYSW, K5 KEYSW, K50 KEYSW, K51 KEYSW, K52 KEYSW, K53 KEYSW, K54 KEYSW, K55 KEYSW, K56 KEYSW, K57 KEYSW, K58 KEYSW, K59 KEYSW, K6 KEYSW, K60 KEYSW, K61 KEYSW, K62 KEYSW, K63 KEYSW, K64 KEYSW, K65 KEYSW, K7 KEYSW, K9 KEYSW, U0 ProMicro, U1 74HC595

Commit message: added screw holes, positioned switches on pcb
Parts:
- added  : , Button_Switch_Keyboard:SW_Cherry_MX_6.25u_Stabs, F.Cu at (131.2, 85.3)
- added Poker_oval_hole: VAL**, keyboard_parts:Poker_oval_hole, F.Cu at (128.2, 47.0)
- added Poker_oval_hole: VAL**, keyboard_parts:Poker_oval_hole, F.Cu at (190.5, 85.2)
- added Poker_oval_hole: VAL**, keyboard_parts:Poker_oval_hole, F.Cu at (259.8, 27.9)
- added Poker_side_edge_long: VAL**, keyboard_parts:Poker_side_edge_long, F.Cu at (285.6, 58.0)
- added Poker_side_edge_long: VAL**, keyboard_parts:Poker_side_edge_long, F.Cu at (-0.60, 57.9)
- added REF**: MountingHole_2.2mm_M2, MountingHole:MountingHole_2.2mm_M2, F.Cu at (25.2, 27.9)
- K0, K1, K10, K11, K12, K13, K14, K15, K16, K17, K18, K19, K2, K20, K21, K22, K23, K24, K25, K26, K27, K28, K29, K3, K30, K31, K32, K33, K34, K35, K36, K37, K38, K39, K4, K41, K42, K43, K44, K45, K46, K47, K48, K49, K5, K50, K51, K52, K53, K54, K55, K56, K57, K58, K6, K60, K61, K62, K63, K64, K65, K7, K9: footprint Button_Switch_Keyboard:SW_Cherry_MX_1.00u_PCB -> kalih keyswitches:Kailh_socket
- K40: footprint Button_Switch_Keyboard:SW_Cherry_MX_ISOEnter_PCB -> kalih keyswitches:Kailh_socket
- K59: footprint Button_Switch_Keyboard:SW_Cherry_MX_6.25u_PCB -> kalih keyswitches:Kailh_socket
- moved U0 183.6 mm to (136.0, 145.4)
- moved U1 102.7 mm to (129.9, 172.6), turned to 0 degrees
- moved K50 5.23 mm to (162.2, 66.3)
- moved K52 5.23 mm to (200.3, 66.3)
- moved K53 5.23 mm to (219.3, 66.3)
- moved K56 5.23 mm to (276.5, 66.3)
- moved K60 5.23 mm to (200.3, 85.3)
- moved K61 5.23 mm to (219.3, 85.3)
- moved K64 5.23 mm to (276.5, 85.3)
- moved K21 5.23 mm to (95.5, 28.2)
- moved K24 5.23 mm to (152.6, 28.2)
- moved K33 5.23 mm to (162.2, 9.14)
- moved K35 5.23 mm to (200.3, 9.14)
- moved K36 5.23 mm to (219.3, 9.14)
- moved K38 5.23 mm to (266.9, 9.14)
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Connections:
- U0 pad 1: Net-(U0-Pad1) -> (no net)
- U0 pad 16: Net-(U0-Pad16) -> (no net)
- U0 pad 2: Net-(U0-Pad2) -> (no net)
- U0 pad 20: Net-(U0-Pad20) -> (no net)
- U0 pad 22: Net-(U0-Pad22) -> (no net)
- U0 pad 24: Net-(U0-Pad24) -> (no net)
- U0 pad 5: Net-(U0-Pad5) -> (no net)
- U0 pad 6: Net-(U0-Pad6) -> (no net)
- U1 pad 9: Net-(U1-Pad9) -> (no net)

Commit message: changed circuit to 5x13, designed pcb
Parts:
- added REF**: SW_Stabilizer, kalih keyswitches:MX_Stabilizer_2u, F.Cu at (274.1, 37.8)
-  : renamed from REF**
- moved U0 167.3 mm to (39.0, 9.12), turned to 0 degrees
- moved U1 100.8 mm to (169.4, 79.8), turned to 270 degrees
- moved D65 22.8 mm to (269.6, 75.8), turned to 0 degrees
- moved D1 14.2 mm to (24.8, 19.9), turned to 0 degrees
- moved D56 8.96 mm to (277.6, 75.8), turned to 0 degrees
- moved D17 5.18 mm to (29.0, 33.0), turned to 180 degrees
- moved D14 3.41 mm to (128.8, 57.0)
- moved D39 2.25 mm to (257.4, 36.8)
- moved D55 1.19 mm to (266.9, 71.7)
Connections:
- D10 pad 1: row1 -> row2
- D11 pad 1: row1 -> row2
- D12 pad 1: row1 -> row2
- D13 pad 1: row1 -> row2
- D14 pad 1: row1 -> row2
- D15 pad 1: row1 -> row2
- D16 pad 1: row1 -> row2
- D17 pad 1: row2 -> row1
- D18 pad 1: row2 -> row1
- D19 pad 1: row2 -> row1
- D20 pad 1: row2 -> row1
- D21 pad 1: row2 -> row1
- D22 pad 1: row2 -> row1
- D23 pad 1: row2 -> row1
- D24 pad 1: row2 -> row1
- D33 pad 1: row4 -> row0
- D34 pad 1: row4 -> row0
- D35 pad 1: row4 -> row0
- D36 pad 1: row4 -> row0
- D37 pad 1: row4 -> row0
- D38 pad 1: row4 -> row0
- D39 pad 1: row4 -> row1
- D40 pad 1: row4 -> row1
- D41 pad 1: row5 -> row1
- D42 pad 1: row5 -> row1
- D43 pad 1: row5 -> row1
- D44 pad 1: row5 -> row1
- D45 pad 1: row5 -> row2
- D46 pad 1: row5 -> row2
- D47 pad 1: row5 -> row2
- D48 pad 1: row5 -> row2
- D49 pad 1: row6 -> row2
- D50 pad 1: row6 -> row3
- D51 pad 1: row6 -> row3
- D52 pad 1: row6 -> row3
- D53 pad 1: row6 -> row3
- D54 pad 1: row6 -> row3
- D55 pad 1: row6 -> row3
- D56 pad 1: row6 -> row2
- D57 pad 1: row7 -> row4
- D59 pad 1: row7 -> row4
- D60 pad 1: row7 -> row4
- D61 pad 1: row7 -> row4
- D62 pad 1: row7 -> row4
- D63 pad 1: row7 -> row4
- D64 pad 1: row7 -> row4
- D65 pad 1: row7 -> row4
- D66 pad 1: row8 -> row4
- D9 pad 1: row1 -> row2
- K33 pad 2: col0 -> col8
- K34 pad 2: col1 -> col9
- K35 pad 2: col2 -> col10
- K36 pad 2: col3 -> col11
- K37 pad 2: col4 -> col12
- K38 pad 2: col5 -> col13
- K39 pad 2: col6 -> col12
- K40 pad 2: col7 -> col13
- K41 pad 2: col0 -> col8
- K42 pad 2: col1 -> col9
- K43 pad 2: col2 -> col10
- K44 pad 2: col3 -> col11
- K45 pad 2: col4 -> col9
- K46 pad 2: col5 -> col10
- K47 pad 2: col6 -> col11
- K48 pad 2: col7 -> col12
- K49 pad 2: col0 -> col8
- K50 pad 2: col1 -> col8
- K51 pad 2: col2 -> col9
- K52 pad 2: col3 -> col10
- K53 pad 2: col4 -> col11
- K54 pad 2: col5 -> col12
- K55 pad 2: col6 -> col13
- K56 pad 2: col7 -> col13
- K57 pad 2: col0 -> col1
- K58 pad 2: col1 -> col2
- K59 pad 2: col2 -> col3
- K60 pad 2: col3 -> col9
- K61 pad 2: col4 -> col10
- K62 pad 2: col5 -> col11
- K63 pad 2: col6 -> col12
- K64 pad 2: col7 -> col13
- U0 pad 1: (no net) -> Net-(U0-Pad1)
- U0 pad 12: row5 -> col5
- U0 pad 13: row6 -> latch
- U0 pad 14: row7 -> clock
- U0 pad 15: row8 -> data
- U0 pad 16: (no net) -> col0
- U0 pad 17: latch -> col1
- U0 pad 18: clock -> col2
- U0 pad 19: data -> col3
- U0 pad 2: (no net) -> Net-(U0-Pad2)
- U0 pad 20: (no net) -> col4
- U0 pad 22: (no net) -> Net-(U0-Pad22)
- U0 pad 24: (no net) -> Net-(U0-Pad24)
- U0 pad 5: (no net) -> Net-(U0-Pad5)
- U0 pad 6: (no net) -> Net-(U0-Pad6)
- U1 pad 1: col1 -> col12
- U1 pad 15: col0 -> col13
- U1 pad 2: col2 -> col11
- U1 pad 3: col3 -> col10
- U1 pad 4: col4 -> col9
- U1 pad 5: col5 -> col8
- U1 pad 6: col6 -> col7
- U1 pad 7: col7 -> col6
- U1 pad 9: (no net) -> Net-(U1-Pad9)
Routing:
- net row1: track 0.00 -> 376.1 mm
- net row4: track 0.00 -> 354.6 mm
- net row3: track 0.00 -> 346.9 mm
- net row2: track 0.00 -> 344.8 mm
- net row0: track 0.00 -> 280.2 mm
- net data: track 0.00 -> 259.9 mm
- net clock: track 0.00 -> 250.5 mm
- net latch: track 0.00 -> 244.2 mm
- net col5: track 0.00 -> 242.2 mm
- net GND: track 0.00 -> 218.2 mm
- net col13: track 0.00 -> 215.2 mm
- net col12: track 0.00 -> 189.7 mm
- net col3: track 0.00 -> 177.0 mm
- net col11: track 0.00 -> 174.8 mm
- net col10: track 0.00 -> 158.3 mm
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- added copper zone on B.Cu, net GND
- added copper zone on F.Cu, net VCC

Commit message: flipped arduino to other side
Parts:
- U0: moved to B.Cu
Connections:
- U0 pad 10: row3 -> col3
- U0 pad 11: row4 -> row0
- U0 pad 13: latch -> data
- U0 pad 15: data -> latch
- U0 pad 18: col2 -> row2
- U0 pad 19: col3 -> row3
- U0 pad 20: col4 -> row1
- U0 pad 7: row0 -> row4
- U0 pad 8: row1 -> col2
- U0 pad 9: row2 -> col4
Routing:
- net GND: track 218.2 -> 0.00 mm
- net row3: track 346.9 -> 547.7 mm
- net col3: track 177.0 -> 272.3 mm
- net row2: track 344.8 -> 315.1 mm
- net row1: track 376.1 -> 349.0 mm
- net col1: track 128.9 -> 103.4 mm
- net data: track 259.9 -> 239.9 mm
- net row4: track 354.6 -> 374.6 mm
- net Net-(D1-Pad2): track 32.0 -> 17.9 mm
- net clock: track 250.5 -> 237.6 mm
- net col5: track 242.2 -> 253.1 mm
- net col0: track 124.6 -> 133.7 mm
- net latch: track 244.2 -> 235.7 mm
- net col4: track 121.5 -> 116.4 mm
- net row0: track 280.2 -> 279.7 mm
