File: kicad/keyboard2/keyboard.kicad_pcb (KiCad board)
At the start: 2 copper layers, 285 x 94.6 mm, 140 parts, among them K0 KEYSW, K1 KEYSW, K10 KEYSW, K11 KEYSW, K12 KEYSW, K13 KEYSW, K14 KEYSW, K15 KEYSW, K16 KEYSW, K17 KEYSW, K18 KEYSW, K19 KEYSW, K2 KEYSW, K20 KEYSW, K21 KEYSW, K22 KEYSW, K23 KEYSW, K24 KEYSW, K25 KEYSW, K26 KEYSW, K27 KEYSW, K28 KEYSW, K29 KEYSW, K3 KEYSW, K30 KEYSW, K31 KEYSW, K32 KEYSW, K33 KEYSW, K34 KEYSW, K35 KEYSW, K36 KEYSW, K37 KEYSW, K38 KEYSW, K39 KEYSW, K4 KEYSW, K40 KEYSW, K41 KEYSW, K42 KEYSW, K43 KEYSW, K44 KEYSW, K45 KEYSW, K46 KEYSW, K47 KEYSW, K48 KEYSW, K49 KEYSW, K5 KEYSW, K50 KEYSW, K51 KEYSW, K52 KEYSW, K53 KEYSW, K54 KEYSW, K55 KEYSW, K56 KEYSW, K57 KEYSW, K58 KEYSW, K59 KEYSW, K6 KEYSW, K60 KEYSW, K61 KEYSW, K62 KEYSW, K63 KEYSW, K64 KEYSW, K65 KEYSW, K7 KEYSW, K9 KEYSW, U0 ProMicro, U1 74HC595

Commit message: completed main layout
Parts:
- removed  : , Button_Switch_Keyboard:SW_Cherry_MX_6.25u_Stabs
- removed  : MountingHole_2.2mm_M2, MountingHole:MountingHole_2.2mm_M2
- removed the Poker_side_edge_long at (285.6, 58.0)
- removed the Poker_side_edge_long at (-0.60, 57.9)
- removed the REF** at (274.1, 37.8)
- removed U1: 74HC595, Package_DIP:DIP-16_W7.62mm
- added C0: 22pf, Capacitor_SMD:C_1206_3216Metric_Pad1.42x1.75mm_HandSolder, B.Cu at (81.5, 82.2)
- added C1: 22pf, Capacitor_SMD:C_1206_3216Metric_Pad1.42x1.75mm_HandSolder, B.Cu at (81.5, 84.8)
- added C2: 1uf, Capacitor_SMD:C_1206_3216Metric_Pad1.42x1.75mm_HandSolder, B.Cu at (99.6, 75.6)
- added J1: USB_B_Micro, keyboard_parts:USB_microB, B.Cu at (18.2, 1.44)
- added JP0: , Button_Switch_THT:SW_DIP_SPSTx01_Slide_6.7x4.1mm_W7.62mm_P2.54mm_LowProfile, F.Cu at (29.1, 52.0)
- added Poker_oval_hole: VAL**, keyboard_parts:Poker_oval_hole, F.Cu at (25.2, 27.9)
- added Poker_side_edge_long: VAL**, keyboard_parts:Poker_side_edge_long, F.Cu at (0.00, 56.5)
- added Poker_side_edge_long: VAL**, keyboard_parts:Poker_side_edge_long, F.Cu at (285.0, 56.5)
- added R0: 22, Resistor_SMD:R_1206_3216Metric_Pad1.42x1.75mm_HandSolder, B.Cu at (97.3, 93.0)
- added R1: 22, Resistor_SMD:R_1206_3216Metric_Pad1.42x1.75mm_HandSolder, B.Cu at (102.8, 93.0)
- added R2: 10k, Resistor_SMD:R_1206_3216Metric_Pad1.42x1.75mm_HandSolder, B.Cu at (81.5, 87.4)
- added REF**: SW_Stabilizer, kalih keyswitches:MX_Stabilizer_2u, F.Cu at (274.1, 37.7)
- added REF**: SW_Stabilizer, kalih keyswitches:MX_Stabilizer_2u, F.Cu at (266.9, 9.14)
- added REF**: SW_Cherry_MX_6.25u_Stabs, Button_Switch_Keyboard:SW_Cherry_MX_6.25u_Stabs, F.Cu at (131.2, 85.3)
- added Y0: 16 MHZ, Crystal:Crystal_SMD_Abracon_ABM3-2Pin_5.0x3.2mm_HandSoldering, B.Cu at (88.0, 84.8)
- U0: value ProMicro -> ATmega32U4-AU; footprint keebs:Pro_Micro -> Package_QFP:TQFP-44_10x10mm_P0.8mm
- moved U0 96.0 mm to (98.0, 84.8), turned to 90 degrees
- moved D1 14.2 mm to (38.4, 15.5), turned to 90 degrees
- moved D40 9.92 mm to (274.2, 47.2), turned to 0 degrees
- moved D9 5.50 mm to (31.7, 55.2), turned to 180 degrees
- moved D17 1.67 mm to (29.0, 34.7)
- moved D38 1.50 mm to (276.5, 14.0)
- moved D55 0.95 mm to (267.0, 72.6)
- moved Poker_oval_hole 0.25 mm to (260.1, 27.9)
- turned K0 to 90 degrees
- turned K15 to 90 degrees
Connections:
- U0 pad 10: col3 -> col5
- U0 pad 11: row0 -> col6
- U0 pad 12: col5 -> row4
- U0 pad 13: data -> Reset
- U0 pad 14: clock -> VCC
- U0 pad 15: latch -> Earth
- U0 pad 16: col0 -> Net-(C1-Pad1)
- U0 pad 17: col1 -> Net-(C0-Pad1)
- U0 pad 18: row2 -> Net-(U0-Pad18)
- U0 pad 19: row3 -> col13
- U0 pad 2: Net-(U0-Pad2) -> VCC
- U0 pad 20: row1 -> col12
- U0 pad 21: VCC -> col11
- U0 pad 22: Net-(U0-Pad22) -> col9
- U0 pad 23: GND -> Earth
- U0 pad 24: Net-(U0-Pad24) -> VCC
- U0 pad 3: GND -> USBD-
- U0 pad 4: GND -> USBD+
- U0 pad 5: Net-(U0-Pad5) -> Earth
- U0 pad 7: row4 -> VCC
- U0 pad 8: col2 -> col3
Routing:
- net row3: track 547.7 -> 247.7 mm
- net data: track 239.9 -> 0.00 mm
- net clock: track 237.6 -> 0.00 mm
- net latch: track 235.7 -> 0.00 mm
- net col3: track 272.3 -> 69.0 mm
- net col5: track 253.1 -> 69.0 mm
- net col13: track 215.2 -> 102.8 mm
- net row4: track 374.6 -> 263.3 mm
- net row1: track 349.0 -> 251.3 mm
- net col12: track 189.7 -> 97.9 mm
- net col11: track 174.8 -> 97.9 mm
- net row2: track 315.1 -> 245.1 mm
- net col0: track 133.7 -> 71.2 mm
- net col10: track 158.3 -> 97.9 mm
- net col4: track 116.4 -> 69.0 mm
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- added copper zone on B.Cu, net Earth
- removed copper zone on B.Cu, net GND

Commit message: Completed first attempt at keyboard2 tracks
Parts:
- moved R0 20.0 mm to (116.9, 88.7), turned to 90 degrees
- moved C2 18.7 mm to (109.1, 91.7)
- moved R1 17.2 mm to (119.4, 88.7), turned to 90 degrees
- moved U0 9.80 mm to (107.6, 82.9)
- moved Y0 9.80 mm to (97.6, 82.9)
- moved C0 9.80 mm to (91.1, 80.3)
- moved C1 9.80 mm to (91.1, 82.9)
- moved R2 9.80 mm to (91.1, 85.4)
- moved D60 3.76 mm to (140.7, 87.9)
Connections:
- K59 pad 2: col3 -> col8
- U0 pad 10: col5 -> col13
- U0 pad 11: col6 -> col3
- U0 pad 19: col13 -> col0
- U0 pad 20: col12 -> col1
- U0 pad 21: col11 -> col2
- U0 pad 22: col9 -> col4
- U0 pad 25: col10 -> col5
- U0 pad 26: col8 -> row2
- U0 pad 27: col7 -> row1
- U0 pad 28: col2 -> row3
- U0 pad 29: col1 -> row0
- U0 pad 30: col0 -> col6
- U0 pad 31: row3 -> col7
- U0 pad 32: row2 -> col8
- U0 pad 36: row0 -> col9
- U0 pad 37: row1 -> col10
- U0 pad 8: col3 -> col11
- U0 pad 9: col4 -> col12
Routing:
- net Net-(J1-Pad3): track 6.68 -> 186.8 mm, vias 0 -> 2
- net Net-(J1-Pad2): track 6.02 -> 185.2 mm, vias 0 -> 2
- net col13: track 102.8 -> 278.1 mm
- net col12: track 97.9 -> 253.0 mm
- net col11: track 97.9 -> 232.9 mm
- net Reset: track 10.9 -> 132.3 mm, vias 0 -> 1
- net col0: track 71.2 -> 182.8 mm
- net col10: track 97.9 -> 207.8 mm
- net col1: track 97.8 -> 184.9 mm
- net col9: track 97.1 -> 183.3 mm
- net row0: track 257.8 -> 335.2 mm
- net col3: track 69.0 -> 137.9 mm, vias 0 -> 2
- net col8: track 69.0 -> 134.5 mm
- net col2: track 93.9 -> 151.6 mm
- net row1: track 251.3 -> 301.8 mm
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